Commit message: edit

File: stickman/stickman.urdf (robot description, URDF)
Before this commit: robot stickman, 5 links, 4 joints
Joints:
- joint left_hip: origin xyz=0.05 0 -0.2 rpy=0 0 0 -> xyz=0.1 0 -0.2 rpy=0 0 0
- joint right_hip: origin xyz=-0.05 0 -0.2 rpy=0 0 0 -> xyz=-0.1 0 -0.2 rpy=0 0 0
